Commit message: Add task: DroneAgent

File: assets/urdf/cube.urdf (robot description, URDF)
Before this commit: robot object, 1 links, 0 joints
Links:
- link object: geometry collision box size=0.5 0.5 0.5; visual box size=0.5 0.5 0.5

File: assets/urdf/cube02.urdf (robot description, URDF)
Before this commit: robot cartpole, 3 links, 2 joints
Joints:
- joint cart_to_pole: origin xyz=0.12 0 0 -> xyz=0.0 0 0
